File: antenna-board.kicad_pcb (KiCad board)
At the start: 2 copper layers, 42.4 x 42.4 mm, 2 parts, among them J1 Conn_01x01, U1 U.FLport

Commit message: Fixed Things
Routing:
- net GNDREF: track 415.0 -> 447.4 mm, vias 89 -> 97
- net DATA: track 0.00 -> 9.40 mm
Other:
- board text added: "SFU Rocketry Antenna GND Plane REV 1b"
- board text removed: "SFU Rocketry Antenna GND Plane REV 1a"
Changed lines of the file:
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@@
     (thickness 1.6)
     (drawings 2)
-    (tracks 253)
+    (tracks 277)
     (zones 0)
     (modules 2)
@@
   (layers
     (0 F.Cu signal)
-    (31 B.Cu signal)
+    (31 B.Cu signal hide)
     (32 B.Adhes user)
     (33 F.Adhes user)
@@
       (net 1 DATA))
   )
-  (gr_text "SFU Rocketry\nAntenna GND Plane\nREV 1a\n" (at 100.11 93.29) (layer F.SilkS)
+  (gr_text "SFU Rocketry\nAntenna GND Plane\nREV 1b\n\n" (at 100.11 93.29) (layer F.SilkS)
     (effects (font (size 0.7 0.7) (thickness 0.15)))
   )
   (gr_circle (center 100 100) (end 115 115) (layer Edge.Cuts) (width 0.2))
+  (segment (start 100 101.6) (end 100 111) (width 1.2) (layer F.Cu) (net 1))
+  (segment (start 109.22 94.615) (end 107.605 94.615) (width 0.25) (layer F.Cu) (net 2))
+  (segment (start 107.605 94.615) (end 105.69 92.7) (width 0.25) (layer F.Cu) (net 2))
+  (via (at 105.69 92.7) (size 0.6) (drill 0.4) (layers F.Cu B.Cu) (net 2))
+  (segment (start 111.76 95.885) (end 111.76 96.88) (width 0.25) (layer F.Cu) (net 2))
+  (segment (start 111.76 96.88) (end 109.01 99.63) (width 0.25) (layer F.Cu) (net 2))
+  (via (at 109.01 99.63) (size 0.6) (drill 0.4) (layers F.Cu B.Cu) (net 2))
+  (segment (start 103.505 85.725) (end 101.725 85.725) (width 0.25) (layer F.Cu) (net 2))
+  (segment (start 101.725 85.725) (end 98.73 88.72) (width 0.25) (layer F.Cu) (net 2))
+  (via (at 98.73 88.72) (size 0.6) (drill 0.4) (layers F.Cu B.Cu) (net 2))
+  (segment (start 95 94) (end 95 98.35) (width 0.25) (layer F.Cu) (net 2))
+  (segment (start 95 98.35) (end 92.57 100.78) (width 0.25) (layer F.Cu) (net 2))
+  (via (at 92.57 100.78) (size 0.6) (drill 0.4) (layers F.Cu B.Cu) (net 2))
+  (segment (start 93 94) (end 93 95.34) (width 0.25) (layer F.Cu) (net 2))
+  (segment (start 93 95.34) (end 90.25 98.09) (width 0.25) (layer F.Cu) (net 2))
+  (via (at 90.25 98.09) (size 0.6) (drill 0.4) (layers F.Cu B.Cu) (net 2))
+  (segment (start 101 98) (end 103 98) (width 0.25) (layer F.Cu) (net 2))
+  (via (at 103 98) (size 0.6) (drill 0.4) (layers F.Cu B.Cu) (net 2))
+  (segment (start 97 98) (end 97 101.06) (width 0.25) (layer F.Cu) (net 2))
+  (segment (start 97 101.06) (end 97 102.08) (width 0.25) (layer F.Cu) (net 2))
+  (segment (start 97 100) (end 97 101.06) (width 0.25) (layer F.Cu) (net 2))
+  (via (at 97 101.06) (size 0.6) (drill 0.4) (layers F.Cu B.Cu) (net 2))
+  (segment (start 103 100) (end 103 101.02) (width 0.25) (layer F.Cu) (net 2))
+  (segment (start 103 101.02) (end 102.91 101.11) (width 0.25) (layer F.Cu) (net 2))
+  (via (at 102.91 101.11) (size 0.6) (drill 0.4) (layers F.Cu B.Cu) (net 2))
+  (segment (start 102.87 102.235) (end 102.87 103.505) (width 0.25) (layer F.Cu) (net 2))
+  (via (at 102.87 103.505) (size 0.6) (drill 0.4) (layers F.Cu B.Cu) (net 2))
   (segment (start 104.775 112.395) (end 108.585 112.395) (width 0.25) (layer F.Cu) (net 2))
   (segment (start 108.585 112.395) (end 111.125 112.395) (width 0.25) (layer F.Cu) (net 2))
@@
   (via (at 97.155 103.505) (size 0.6) (drill 0.4) (layers F.Cu B.Cu) (net 2))
   (segment (start 97.155 102.235) (end 97.155 103.505) (width 0.25) (layer F.Cu) (net 2))
-  (segment (start 97 98) (end 97 102.08) (width 0.25) (layer F.Cu) (net 2))
   (segment (start 97 102.08) (end 97.155 102.235) (width 0.25) (layer F.Cu) (net 2))
   (via (at 97.155 102.235) (size 0.6) (drill 0.4) (layers F.Cu B.Cu) (net 2))
@@
   (segment (start 102.87 103.505) (end 102.87 104.775) (width 0.25) (layer F.Cu) (net 2))
   (via (at 102.87 104.775) (size 0.6) (drill 0.4) (layers F.Cu B.Cu) (net 2))
-  (via (at 102.87 103.505) (size 0.6) (drill 0.4) (layers F.Cu B.Cu) (net 2))
-  (segment (start 102.87 102.235) (end 102.87 103.505) (width 0.25) (layer F.Cu) (net 2))
   (segment (start 103 102.105) (end 102.87 102.235) (width 0.25) (layer F.Cu) (net 2))
   (via (at 102.87 102.235) (size 0.6) (drill 0.4) (layers F.Cu B.Cu) (net 2))
@@
     (connect_pads yes (clearance 0.2))
     (min_thickness 0.2)
-    (fill yes (arc_segments 16) (thermal_gap 0.508) (thermal_bridge_width 0.508))
+    (fill (arc_segments 16) (thermal_gap 0.508) (thermal_bridge_width 0.508))
     (polygon
       (pts
@@
     (connect_pads yes (clearance 0.2))
     (min_thickness 0.2)
-    (fill yes (arc_segments 16) (thermal_gap 0.508) (thermal_bridge_width 0.508))
+    (fill (arc_segments 16) (thermal_gap 0.508) (thermal_bridge_width 0.508))
     (polygon
       (pts
@@
     (priority 11)
     (connect_pads yes (clearance 0.2))
-    (min_thickness 1.2)
-    (fill yes (arc_segments 16) (thermal_gap 0.508) (thermal_bridge_width 0.508))
+    (min_thickness 0.258)
+    (fill (arc_segments 16) (thermal_gap 0.508) (thermal_bridge_width 0.508))
     (polygon
       (pts
-        (xy 100.75 100.8) (xy 100.75 112.43) (xy 99.25 112.43) (xy 99.25 100.8)
-      )
-    )
-  )
-  (zone (net 0) (net_name "") (layer F.Cu) (hatch full 0.508)
-    (connect_pads yes (clearance 0.2))
-    (min_thickness 1.2)
-    (keepout (tracks not_allowed) (vias not_allowed) (copperpour not_allowed))
-    (fill yes (arc_segments 16) (thermal_gap 0.508) (thermal_bridge_width 0.508))
-    (polygon
-      (pts
-        (xy 97.79 101.670252) (xy 99.06 101.670252) (xy 99.0346 112.5982) (xy 97.7746 112.5982)
+        (xy 100.6 100.85) (xy 100.6 112.4) (xy 99.4 112.4) (xy 99.4 100.85)
       )
     )
@@
     (polygon
       (pts
-        (xy 100.965 101.6) (xy 102.235 101.6) (xy 102.235 112.6236) (xy 100.965 112.6236)
+        (xy 97.8 101.7) (xy 99.2 101.7) (xy 99.2 112.6) (xy 97.79 112.6)
       )
     )
+  )
+  (zone (net 0) (net_name "") (layer F.Cu) (hatch full 0.508)
+    (connect_pads yes (clearance 0.2))
+    (min_thickness 1.2)
+    (keepout (tracks not_allowed) (vias not_allowed) (copperpour not_allowed))
+    (fill (arc_segments 16) (thermal_gap 0.508) (thermal_bridge_width 0.508))
+    (polygon
+      (pts
+        (xy 100.8 101.6) (xy 102.2 101.6) (xy 102.2 112.6) (xy 100.8 112.6)
+      )
+    )

Commit message: Fixed Vias
Routing:
- net GNDREF: track 447.4 -> 508.9 mm, vias 97 -> 114
